Commit message: fix mic position

File: rb1_description/urdf/sensors/mic_array.urdf.xacro (robot description, xacro)
@@ -3,5 +3,5 @@
     <xacro:macro name="mic_array" params="name parent">
         <joint name="${name}_joint" type="fixed">
-            <origin xyz="0.0 0.06 0.05" rpy="0.0 0.0 0.0"/>
+            <origin xyz="0.0 0.02 0.07" rpy="0.0 0.0 0.0"/>
             <parent link="${parent}"/>
             <child link="${name}_link"/>
